Commit message: set up urdf/srdf files for collision checking

File: workspace/src/par_pkg/urdf/arm-with-gripper.urdf.xacro (robot description, xacro)
@@ -5,15 +5,22 @@
     <xacro:include filename="$(find ur_description)/urdf/ur.urdf.xacro"/>
     <xacro:include filename="onrobot_rg2_model.urdf"/>
+    <xacro:include filename="onrobot_quick_changer_model.urdf"/>
     <xacro:include filename="onrobot_eyes_model.urdf"/>
     <xacro:macro name="ur" params="name ur_type"/>
     <joint name="eyes_joint" type="fixed">
-        <origin rpy="0 0 0" xyz="0 0 0"/>
+        <origin rpy="0 0 3.1416" xyz="0 0 0"/>
         <parent link="tool0"/>
         <child link="onrobot_eyes_base_link"/>
         <axis xyz="0 0 0"/>
     </joint>
+    <joint name="quick_changer_joint" type="fixed">
+        <origin rpy="0 0 1.5708" xyz="0 0 0"/>
+        <parent link="onrobot_eyes_tool_link"/>
+        <child link="onrobot_quick_changer_base_link"/>
+        <axis xyz="0 0 0"/>
+    </joint>
     <joint name="gripper_joint" type="fixed">
         <origin rpy="0 0 0" xyz="0 0 0"/>
-        <parent link="onrobot_eyes_base_link"/>
+        <parent link="onrobot_quick_changer_tool_link"/>
         <child link="onrobot_rg2_base_link"/>
         <axis xyz="0 0 0"/>

File: workspace/src/par_pkg/urdf/onrobot_quick_changer_model.urdf (robot description, URDF)
Before this commit: robot onrobot_eyes_model, 2 links, 1 joints
Links:
- removed link onrobot_eyes_base_link
- removed link onrobot_eyes_tool_link
- added link onrobot_quick_changer_base_link, mass 0.06; collision mesh filename=package://par_pkg/meshes/collision/quick_changer.stl; visual mesh filename=package://par_pkg/meshes/visual/quick_changer.stl
- added link onrobot_quick_changer_tool_link
Joints:
- removed joint onrobot_eyes_joint
- added joint onrobot_quick_changer_joint: type fixed, parent onrobot_quick_changer_base_link, child onrobot_quick_changer_tool_link, origin xyz=0 0 0.0021 rpy=0 0 0, axis 0 0 0
