Commit message: Fixed measurements

File: workspace/src/par_pkg/urdf/onrobot_eyes_model.urdf (robot description, URDF)
Before this commit: robot onrobot_eyes_model, 2 links, 1 joints
Joints:
- joint onrobot_eyes_joint: origin xyz=0 0 0.012 rpy=0 0 0 -> xyz=0 0 0.0105 rpy=0 0 0

Commit message: started updating cameralink

File: workspace/src/par_pkg/urdf/onrobot_eyes_model.urdf (robot description, URDF)
Before this commit: robot onrobot_eyes_model, 2 links, 1 joints
Links:
- added link camera_link
Joints:
- added joint camera_joint: type fixed, parent onrobot_eyes_base_link, child camera_link, origin xyz=0 0 0.105 rpy=0 0 0, axis 0 0 0

Commit message: Moved camera position to y axis

File: workspace/src/par_pkg/urdf/onrobot_eyes_model.urdf (robot description, URDF)
Before this commit: robot onrobot_eyes_model, 3 links, 2 joints
Joints:
- joint camera_joint: origin xyz=0 0 0.105 rpy=0 0 0 -> xyz=0 0.105 0 rpy=0 0 0
