Commit message: Added all the new urdfs

File: workspace/src/par_pkg/urdf/onrobot_rg2_gripper.urdf (robot description, URDF)
Before this commit: robot onrobot_rg2_gripper, 7 links, 6 joints
Links:
- link left_finger: geometry collision mesh filename=package://par_pkg/meshes/collision/rg2_finger.stl; visual mesh filename=package://par_pkg/meshes/visual/rg2_finger.dae
- link left_inner_knuckle: geometry collision mesh filename=package://par_pkg/meshes/collision/rg2_inner_knuckle.stl; visual mesh filename=package://par_pkg/meshes/visual/rg2_inner_knuckle.dae
- link left_outer_knuckle: geometry collision mesh filename=package://par_pkg/meshes/collision/rg2_outer_knuckle.stl; visual mesh filename=package://par_pkg/meshes/visual/rg2_outer_knuckle.dae
- link onrobot_rg2_base_link: geometry collision mesh filename=package://par_pkg/meshes/collision/rg2_base_link.stl; visual mesh filename=package://par_pkg/meshes/visual/rg2_base_link.dae
- link right_finger: geometry collision mesh filename=package://par_pkg/meshes/collision/rg2_finger.stl; visual mesh filename=package://par_pkg/meshes/visual/rg2_finger.dae
- link right_inner_knuckle: geometry collision mesh filename=package://par_pkg/meshes/collision/rg2_inner_knuckle.stl; visual mesh filename=package://par_pkg/meshes/visual/rg2_inner_knuckle.dae
- link right_outer_knuckle: geometry collision mesh filename=package://par_pkg/meshes/collision/rg2_outer_knuckle.stl; visual mesh filename=package://par_pkg/meshes/visual/rg2_outer_knuckle.dae

Commit message: Added joint limits to grippers

File: workspace/src/par_pkg/urdf/onrobot_rg2_gripper.urdf (robot description, URDF)
Before this commit: robot onrobot_rg2_gripper, 7 links, 6 joints
Joints:
- joint left_finger_joint: limit (none) -> lower=1.875697 upper=3.1069965 effort=1000 velocity=1.0
- joint left_inner_knuckle_joint: limit (none) -> lower=1.875697 upper=3.1069965 effort=1000 velocity=1.0
- joint right_finger_joint: limit (none) -> lower=1.875697 upper=3.1069965 effort=1000 velocity=1.0
- joint right_inner_knuckle_joint: limit (none) -> lower=1.875697 upper=3.1069965 effort=1000 velocity=1.0
- joint right_outer_knuckle_joint: limit (none) -> lower=1.875697 upper=3.1069965 effort=1000 velocity=1.0

Commit message: corrected gripper width to angle function

File: workspace/src/par_pkg/urdf/onrobot_rg2_gripper.urdf (robot description, URDF)
Before this commit: robot onrobot_rg2_gripper, 7 links, 6 joints
Joints:
- joint finger_joint: limit lower=1.875697 upper=3.1069965 effort=1000 velocity=1.0 -> lower=1.87361095202 upper=3.18697121414 effort=1000 velocity=1.0
- joint left_finger_joint: limit lower=1.875697 upper=3.1069965 effort=1000 velocity=1.0 -> lower=1.87361095202 upper=3.18697121414 effort=1000 velocity=1.0
- joint left_inner_knuckle_joint: limit lower=1.875697 upper=3.1069965 effort=1000 velocity=1.0 -> lower=1.87361095202 upper=3.18697121414 effort=1000 velocity=1.0
- joint right_finger_joint: limit lower=1.875697 upper=3.1069965 effort=1000 velocity=1.0 -> lower=1.87361095202 upper=3.18697121414 effort=1000 velocity=1.0
- joint right_inner_knuckle_joint: limit lower=1.875697 upper=3.1069965 effort=1000 velocity=1.0 -> lower=1.87361095202 upper=3.18697121414 effort=1000 velocity=1.0
- joint right_outer_knuckle_joint: limit lower=1.875697 upper=3.1069965 effort=1000 velocity=1.0 -> lower=1.87361095202 upper=3.18697121414 effort=1000 velocity=1.0

Commit message: Started lowering the polycount of the gripper

File: workspace/src/par_pkg/urdf/onrobot_rg2_gripper.urdf (robot description, URDF)
Before this commit: robot onrobot_rg2_gripper, 7 links, 6 joints
Links:
- link left_outer_knuckle: geometry collision mesh filename=package://par_pkg/meshes/collision/rg2_outer_knuckle.stl; visual mesh filename=package://par_pkg/meshes/visual/rg2_outer_knuckle_v2.dae
- link right_outer_knuckle: geometry collision mesh filename=package://par_pkg/meshes/collision/rg2_outer_knuckle.stl; visual mesh filename=package://par_pkg/meshes/visual/rg2_outer_knuckle_v2.dae

Commit message: We now have a lower poly model for the inner and outer knuckles

File: workspace/src/par_pkg/urdf/onrobot_rg2_gripper.urdf (robot description, URDF)
Before this commit: robot onrobot_rg2_gripper, 7 links, 6 joints
Links:
- link left_inner_knuckle: geometry collision mesh filename=package://par_pkg/meshes/collision/rg2_inner_knuckle.stl; visual mesh filename=package://par_pkg/meshes/visual/rg2_inner_knuckle_v2.dae
- link right_inner_knuckle: geometry collision mesh filename=package://par_pkg/meshes/collision/rg2_inner_knuckle.stl; visual mesh filename=package://par_pkg/meshes/visual/rg2_inner_knuckle_v2.dae

Commit message: Finished low poly gripper model

File: workspace/src/par_pkg/urdf/onrobot_rg2_gripper.urdf (robot description, URDF)
Before this commit: robot onrobot_rg2_gripper, 7 links, 6 joints
Links:
- link left_finger: geometry collision mesh filename=package://par_pkg/meshes/collision/rg2_finger.stl; visual mesh filename=package://par_pkg/meshes/visual/rg2_finger_v2.dae
- link onrobot_rg2_base_link: geometry collision mesh filename=package://par_pkg/meshes/collision/rg2_base_link.stl; visual mesh filename=package://par_pkg/meshes/visual/rg2_base_link_v2.dae
- link right_finger: geometry collision mesh filename=package://par_pkg/meshes/collision/rg2_finger.stl; visual mesh filename=package://par_pkg/meshes/visual/rg2_finger_v2.dae
