Commit message: Started setting up urdf for camera

File: workspace/src/par_pkg/urdf/arm-with-camera.urdf.xacro (robot description, xacro)
@@ -6,5 +6,9 @@
     <xacro:include filename="onrobot_quick_changer_model.urdf"/>
     <xacro:include filename="onrobot_eyes_model.urdf"/>
+    <!-- <xacro:include filename="$(find realsense2_description)/urdf/_d415.urdf.xacro"/> -->
     <xacro:macro name="ur" params="name ur_type"/>
+    <!-- <xacro:sensor_d415 parent="on_robot_eyes_base_link" use_nominal_extrinsics="true" add_plug="false" use_mesh="true">
+        <origin xyz="0 0.105 0" rpy="0 0 0"/>
+    </xacro:sensor_d415> -->
     <joint name="eyes_joint" type="fixed">
         <origin rpy="0 0 ${pi}" xyz="0 0 0"/>

Commit message: Added sam's camera link

File: workspace/src/par_pkg/urdf/arm-with-camera.urdf.xacro (robot description, xacro)
@@ -17,4 +17,12 @@
         <origin xyz="-0.000473 0.093319 0.021695" rpy="-${pi/2} -${pi/2} 0"/>
     </xacro:sensor_d415>
+    <!-- This is the camera link provided by Sam, not sure how it was obtained -->
+    <link name="camera_sam_link"/>
+    <joint name="camera_sam_link_joint" type="fixed">
+        <origin rpy="0 -${pi/2} ${pi/2}" xyz="-0.018 -0.11 0.031"/>
+        <parent link="wrist_3_link"/>
+        <child link="camera_sam_link"/>
+        <axis xyz="0 0 0"/>
+    </joint>
     <joint name="eyes_joint" type="fixed">
         <origin rpy="0 0 ${pi}" xyz="0 0 0"/>

Commit message: Added opencv to the docker file, slightly adjusted camera transform

File: workspace/src/par_pkg/urdf/arm-with-camera.urdf.xacro (robot description, xacro)
@@ -15,5 +15,5 @@
             industrial_calibration seems like a good package for doing this.
         -->
-        <origin xyz="-0.000473 0.093319 0.021695" rpy="-${pi/2} -${pi/2} 0"/>
+        <origin xyz="-0.001473 0.093319 0.021695" rpy="-${pi/2} -${pi/2} 0"/>
     </xacro:sensor_d415>
     <!-- This is the camera link provided by Sam, not sure how it was obtained -->

Commit message: sent transform for camera the other way

File: workspace/src/par_pkg/urdf/arm-with-camera.urdf.xacro (robot description, xacro)
@@ -15,5 +15,5 @@
             industrial_calibration seems like a good package for doing this.
         -->
-        <origin xyz="-0.001473 0.093319 0.021695" rpy="-${pi/2} -${pi/2} 0"/>
+        <origin xyz="0.000572 0.093319 0.021695" rpy="-${pi/2} -${pi/2} 0"/>
     </xacro:sensor_d415>
     <!-- This is the camera link provided by Sam, not sure how it was obtained -->

Commit message: Adjusted offset

File: workspace/src/par_pkg/urdf/arm-with-camera.urdf.xacro (robot description, xacro)
@@ -15,5 +15,5 @@
             industrial_calibration seems like a good package for doing this.
         -->
-        <origin xyz="0.000572 0.093319 0.021695" rpy="-${pi/2} -${pi/2} 0"/>
+        <origin xyz="0.684587 0.093319 0.021695" rpy="-${pi/2} -${pi/2} 0"/>
     </xacro:sensor_d415>
     <!-- This is the camera link provided by Sam, not sure how it was obtained -->

Commit message: reconfigured transform to what it was before, awaiting proper calibration

File: workspace/src/par_pkg/urdf/arm-with-camera.urdf.xacro (robot description, xacro)
@@ -15,5 +15,5 @@
             industrial_calibration seems like a good package for doing this.
         -->
-        <origin xyz="0.684587 0.093319 0.021695" rpy="-${pi/2} -${pi/2} 0"/>
+        <origin xyz="-0.000473 0.093319 0.021695" rpy="-${pi/2} -${pi/2} 0"/>
     </xacro:sensor_d415>
     <!-- This is the camera link provided by Sam, not sure how it was obtained -->

Commit message: Tried to fix up camera link

File: workspace/src/par_pkg/urdf/arm-with-camera.urdf.xacro (robot description, xacro)
@@ -15,5 +15,5 @@
             industrial_calibration seems like a good package for doing this.
         -->
-        <origin xyz="-0.000473 0.093319 0.021695" rpy="-${pi/2} -${pi/2} 0"/>
+        <origin xyz="-0.01091 0.105055 0.019792" rpy="-${pi/2} -${pi/2} 0"/>
     </xacro:sensor_d415>
     <!-- This is the camera link provided by Sam, not sure how it was obtained -->

Commit message: fixed malformed urdf

File: workspace/src/par_pkg/urdf/arm-with-camera.urdf.xacro (robot description, xacro)
@@ -1,14 +1,15 @@
 <?xml version="1.0"?>
-<robot xmlns:xacro="http://www.ros.org/wiki/xacro"  name="$(arg name)">
-    <xacro:arg name="name" default="ur"/>
-    <xacro:arg name="ur_type" default="ur5x"/>
-    <xacro:include filename="$(find ur_description)/urdf/ur.urdf.xacro"/>
-    <xacro:include filename="onrobot_quick_changer.urdf"/>
-    <xacro:include filename="onrobot_eyes.urdf"/>
-    <xacro:include filename="$(find realsense2_description)/urdf/_d415.urdf.xacro"/>
+<robot xmlns:xacro="http://www.ros.org/wiki/xacro" name="$(arg name)">
+    <xacro:arg name="name" default="ur" />
+    <xacro:arg name="ur_type" default="ur5x" />
+    <xacro:include filename="$(find ur_description)/urdf/ur.urdf.xacro" />
+    <xacro:include filename="onrobot_quick_changer.urdf" />
+    <xacro:include filename="onrobot_eyes.urdf" />
+    <xacro:include filename="$(find realsense2_description)/urdf/_d415.urdf.xacro" />
     <xacro:property name="plate_depth" value="0.0127" />
-    <xacro:property name="plate_size" value="0.30"/>
-    <xacro:macro name="ur" params="name ur_type"/>
-    <xacro:sensor_d415 parent="onrobot_eyes_base_link" use_nominal_extrinsics="true" add_plug="false" use_mesh="false">
+    <xacro:property name="plate_size" value="0.30" />
+    <xacro:macro name="ur" params="name ur_type" />
+    <xacro:sensor_d415 parent="onrobot_eyes_base_link" use_nominal_extrinsics="true"
+        add_plug="false" use_mesh="false">
         <!--
             These measurements are not 100% accurate, they're the best
@@ -17,50 +18,50 @@
             industrial_calibration seems like a good package for doing this.
         -->
-        <origin xyz="-0.01091 0.105055 0.019792" rpy="-${pi/2} -${pi/2} 0"/>
+        <origin xyz="-0.01091 0.105055 0.019792" rpy="-${pi/2} -${pi/2} 0" />
     </xacro:sensor_d415>
     <!-- This is the camera link provided by Sam, not sure how it was obtained -->
-    <link name="camera_sam_link"/>
+    <link name="camera_sam_link" />
     <joint name="camera_sam_link_joint" type="fixed">
-        <origin rpy="0 -${pi/2} ${pi/2}" xyz="-0.018 -0.11 0.031"/>
-        <parent link="wrist_3_link"/>
-        <child link="camera_sam_link"/>
-        <axis xyz="0 0 0"/>
+        <origin rpy="0 -${pi/2} ${pi/2}" xyz="-0.018 -0.11 0.031" />
+        <parent link="wrist_3_link" />
+        <child link="camera_sam_link" />
+        <axis xyz="0 0 0" />
     </joint>
     <link name="mount_link">
         <visual>
-            <origin xyz="0 0 ${plate_depth/2}"/>
+            <origin xyz="0 0 ${plate_depth/2}" />
             <geometry>
                 <box size="${plate_size} ${plate_size} ${plate_depth}" />
-            <geometry/>
+            </geometry>
         </visual>
         <collision>
-        <origin xyz="0 0 ${plate_depth/2}"/>
+            <origin xyz="0 0 ${plate_depth/2}" />
             <geometry>
                 <box size="${plate_size} ${plate_size} ${plate_depth}" />
-            <geometry/>
+            </geometry>
         </collision>
     </link>
     <joint name="world_joint" type="fixed">
-        <parent link="world"/>
-        <child link="mount_link"/>
-        <axis xyz="0 0 0"/>
+        <parent link="world" />
+        <child link="mount_link" />
+        <axis xyz="0 0 0" />
     </joint>
     <joint name="mount_joint" type="fixed">
-        <origin xyz="0 0 ${plate_depth}"/>
-        <parent link="mount_link"/>
-        <child link="base_link"/>
-        <axis xyz="0 0 0"/>
+        <origin xyz="0 0 ${plate_depth}" />
+        <parent link="mount_link" />
+        <child link="base_link" />
+        <axis xyz="0 0 0" />
     </joint>
     <joint name="eyes_joint" type="fixed">
-        <origin rpy="0 0 ${pi}" xyz="0 0 0"/>
-        <parent link="tool0"/>
-        <child link="onrobot_eyes_base_link"/>
-        <axis xyz="0 0 0"/>
+        <origin rpy="0 0 ${pi}" xyz="0 0 0" />
+        <parent link="tool0" />
+        <child link="onrobot_eyes_base_link" />
+        <axis xyz="0 0 0" />
     </joint>
     <joint name="quick_changer_joint" type="fixed">
-        <origin rpy="0 0 ${pi/2}" xyz="0 0 0"/>
-        <parent link="onrobot_eyes_tool_link"/>
-        <child link="onrobot_quick_changer_base_link"/>
-        <axis xyz="0 0 0"/>
+        <origin rpy="0 0 ${pi/2}" xyz="0 0 0" />
+        <parent link="onrobot_eyes_tool_link" />
+        <child link="onrobot_quick_changer_base_link" />
+        <axis xyz="0 0 0" />
     </joint>
 </robot>

Commit message: Trying to fix robot to mounting plate

File: workspace/src/par_pkg/urdf/arm-with-camera.urdf.xacro (robot description, xacro)
@@ -9,5 +9,5 @@
     <xacro:property name="plate_depth" value="0.0127" />
     <xacro:property name="plate_size" value="0.30" />
-    <xacro:macro name="ur" params="name ur_type" />
+    <xacro:macro name="ur" parent="mount_plate_attach_link" params="name ur_type" />
     <xacro:sensor_d415 parent="onrobot_eyes_base_link" use_nominal_extrinsics="true"
         add_plug="false" use_mesh="false">
@@ -28,5 +28,5 @@
         <axis xyz="0 0 0" />
     </joint>
-    <link name="mount_link">
+    <link name="mount_plate_base_link">
         <visual>
             <origin xyz="0 0 ${plate_depth/2}" />
@@ -42,13 +42,14 @@
         </collision>
     </link>
+    <link name="mount_plate_attach_link"/>
     <joint name="world_joint" type="fixed">
         <parent link="world" />
-        <child link="mount_link" />
+        <child link="mount_plate_base_link" />
         <axis xyz="0 0 0" />
     </joint>
     <joint name="mount_joint" type="fixed">
         <origin xyz="0 0 ${plate_depth}" />
-        <parent link="mount_link" />
-        <child link="base_link" />
+        <parent link="mount_plate_base_link" />
+        <child link="mount_plate_attach_link" />
         <axis xyz="0 0 0" />
     </joint>

Commit message: Fixed xml import maybe

File: workspace/src/par_pkg/urdf/arm-with-camera.urdf.xacro (robot description, xacro)
@@ -9,5 +9,5 @@
     <xacro:property name="plate_depth" value="0.0127" />
     <xacro:property name="plate_size" value="0.30" />
-    <xacro:macro name="ur" parent="mount_plate_attach_link" params="name ur_type" />
+    <xacro:ur_robot name="${name}" parent="mount_plate_attach_link" ur_type="${ur_type}" />
     <xacro:sensor_d415 parent="onrobot_eyes_base_link" use_nominal_extrinsics="true"
         add_plug="false" use_mesh="false">

Commit message: Tried to put mount plate  back in

File: workspace/src/par_pkg/urdf/arm-with-camera.urdf.xacro (robot description, xacro)
@@ -3,5 +3,6 @@
     <xacro:arg name="name" default="ur" />
     <xacro:arg name="ur_type" default="ur5x" />
-    <xacro:include filename="$(find par_pkg)/urdf/ur.urdf.xacro" />
+    <xacro:arg name="parent" default="mount_plate_attach_link"/>
+    <xacro:include filename="$(find ur_description)/urdf/ur.urdf.xacro" />
     <xacro:include filename="onrobot_quick_changer.urdf" />
     <xacro:include filename="onrobot_eyes.urdf" />
@@ -9,5 +10,5 @@
     <xacro:property name="plate_depth" value="0.0127" />
     <xacro:property name="plate_size" value="0.30" />
-    <xacro:ur_robot name="ur" parent="mount_plate_attach_link" />
+    <xacro:macro name="ur" params="name ur_type parent" />
     <xacro:sensor_d415 parent="onrobot_eyes_base_link" use_nominal_extrinsics="true"
         add_plug="false" use_mesh="false">

Commit message: apparently mounted the robot

File: workspace/src/par_pkg/urdf/arm-with-camera.urdf.xacro (robot description, xacro)
@@ -1,14 +1,19 @@
 <?xml version="1.0"?>
 <robot xmlns:xacro="http://www.ros.org/wiki/xacro" name="$(arg name)">
+    <xacro:property name="plate_depth" value="0.0127" />
+    <xacro:property name="plate_size" value="0.30" />
     <xacro:arg name="name" default="ur" />
     <xacro:arg name="ur_type" default="ur5x" />
-    <xacro:arg name="parent" default="mount_plate_attach_link"/>
-    <xacro:include filename="$(find ur_description)/urdf/ur.urdf.xacro" />
+    <xacro:include filename="$(find ur_description)/urdf/ur_macro.xacro" />
     <xacro:include filename="onrobot_quick_changer.urdf" />
     <xacro:include filename="onrobot_eyes.urdf" />
     <xacro:include filename="$(find realsense2_description)/urdf/_d415.urdf.xacro" />
-    <xacro:property name="plate_depth" value="0.0127" />
-    <xacro:property name="plate_size" value="0.30" />
-    <xacro:macro name="ur" params="name ur_type parent" />
+    <xacro:ur_robot
+        name="$(arg name)"
+        ur_type="$(arg ur_type)"
+        parent="mount_plate_attach_link"
+    >
+        <origin xyz="0 0 0"/>
+    </xacro:ur_robot>
     <xacro:sensor_d415 parent="onrobot_eyes_base_link" use_nominal_extrinsics="true"
         add_plug="false" use_mesh="false">
@@ -29,4 +34,5 @@
         <axis xyz="0 0 0" />
     </joint>
+    <link name="mount_plate_attach_link"/>
     <link name="mount_plate_base_link">
         <visual>
@@ -43,10 +49,4 @@
         </collision>
     </link>
-    <link name="mount_plate_attach_link"/>
-    <joint name="world_joint" type="fixed">
-        <parent link="world" />
-        <child link="mount_plate_base_link" />
-        <axis xyz="0 0 0" />
-    </joint>
     <joint name="mount_joint" type="fixed">
         <origin xyz="0 0 ${plate_depth}" />

Commit message: Maybe fixed it

File: workspace/src/par_pkg/urdf/arm-with-camera.urdf.xacro (robot description, xacro)
@@ -43,4 +43,5 @@
         <axis xyz="0 0 0" />
     </joint>
+    <link name="world"/>
     <link name="mount_plate_attach_link"/>
     <link name="mount_plate_base_link">
@@ -58,4 +59,8 @@
         </collision>
     </link>
+    <joint name="world_joint" type="fixed">
+        <parent link="world"/>
+        <child link="mount_plate_base_link"/>
+    </joint>
     <joint name="mount_joint" type="fixed">
         <origin xyz="0 0 ${plate_depth}" />

Commit message: Reverted xacro till I can sort it properly

File: workspace/src/par_pkg/urdf/arm-with-camera.urdf.xacro (robot description, xacro)
@@ -1,30 +1,12 @@
 <?xml version="1.0"?>
-<robot xmlns:xacro="http://www.ros.org/wiki/xacro" name="$(arg name)">
-    <xacro:property name="plate_depth" value="0.0127" />
-    <xacro:property name="plate_size" value="0.30" />
-    <xacro:arg name="name" default="ur" />
-    <xacro:arg name="ur_type" default="ur5x" />
-    <xacro:arg name="tf_prefix" default="" />
-    <xacro:arg name="joint_limit_params" default="$(find ur_description)/config/$(arg ur_type)/joint_limits.yaml"/>
-    <xacro:arg name="kinematics_params" default="$(find ur_description)/config/$(arg ur_type)/default_kinematics.yaml"/>
-    <xacro:arg name="physical_params" default="$(find ur_description)/config/$(arg ur_type)/physical_parameters.yaml"/>
-    <xacro:arg name="visual_params" default="$(find ur_description)/config/$(arg ur_type)/visual_parameters.yaml"/>
-    <xacro:include filename="$(find ur_description)/urdf/ur_macro.xacro" />
-    <xacro:include filename="onrobot_quick_changer.urdf" />
-    <xacro:include filename="onrobot_eyes.urdf" />
-    <xacro:include filename="$(find realsense2_description)/urdf/_d415.urdf.xacro" />
-    <xacro:ur_robot
-        name="$(arg name)"
-        tf_prefix="$(arg tf_prefix)"
-        joint_limits_parameters_file="$(arg joint_limit_params)"
-        kinematics_parameters_file="$(arg kinematics_params)"
-        physical_parameters_file="$(arg physical_params)"
-        visual_parameters_file="$(arg visual_params)"
-        parent="mount_plate_attach_link"
-    >
-        <origin xyz="0 0 0"/>
-    </xacro:ur_robot>
-    <xacro:sensor_d415 parent="onrobot_eyes_base_link" use_nominal_extrinsics="true"
-        add_plug="false" use_mesh="false">
+<robot xmlns:xacro="http://www.ros.org/wiki/xacro"  name="$(arg name)">
+    <xacro:arg name="name" default="ur"/>
+    <xacro:arg name="ur_type" default="ur5x"/>
+    <xacro:include filename="$(find ur_description)/urdf/ur.urdf.xacro"/>
+    <xacro:include filename="onrobot_quick_changer.urdf"/>
+    <xacro:include filename="onrobot_eyes.urdf"/>
+    <xacro:include filename="$(find realsense2_description)/urdf/_d415.urdf.xacro"/>
+    <xacro:macro name="ur" params="name ur_type"/>
+    <xacro:sensor_d415 parent="onrobot_eyes_base_link" use_nominal_extrinsics="true" add_plug="false" use_mesh="false">
         <!--
             These measurements are not 100% accurate, they're the best
@@ -33,51 +15,25 @@
             industrial_calibration seems like a good package for doing this.
         -->
-        <origin xyz="-0.01091 0.105055 0.019792" rpy="-${pi/2} -${pi/2} 0" />
+        <origin xyz="-0.01091 0.105055 0.019792" rpy="-${pi/2} -${pi/2} 0"/>
     </xacro:sensor_d415>
     <!-- This is the camera link provided by Sam, not sure how it was obtained -->
-    <link name="camera_sam_link" />
+    <link name="camera_sam_link"/>
     <joint name="camera_sam_link_joint" type="fixed">
-        <origin rpy="0 -${pi/2} ${pi/2}" xyz="-0.018 -0.11 0.031" />
-        <parent link="wrist_3_link" />
-        <child link="camera_sam_link" />
-        <axis xyz="0 0 0" />
-    </joint>
-    <link name="world"/>
-    <link name="mount_plate_attach_link"/>
-    <link name="mount_plate_base_link">
-        <visual>
-            <origin xyz="0 0 ${plate_depth/2}" />
-            <geometry>
-                <box size="${plate_size} ${plate_size} ${plate_depth}" />
-            </geometry>
-        </visual>
-        <collision>
-            <origin xyz="0 0 ${plate_depth/2}" />
-            <geometry>
-                <box size="${plate_size} ${plate_size} ${plate_depth}" />
-            </geometry>
-        </collision>
-    </link>
-    <joint name="world_joint" type="fixed">
-        <parent link="world"/>
-        <child link="mount_plate_base_link"/>
-    </joint>
-    <joint name="mount_joint" type="fixed">
-        <origin xyz="0 0 ${plate_depth}" />
-        <parent link="mount_plate_base_link" />
-        <child link="mount_plate_attach_link" />
-        <axis xyz="0 0 0" />
+        <origin rpy="0 -${pi/2} ${pi/2}" xyz="-0.018 -0.11 0.031"/>
+        <parent link="wrist_3_link"/>
+        <child link="camera_sam_link"/>
+        <axis xyz="0 0 0"/>
     </joint>
     <joint name="eyes_joint" type="fixed">
-        <origin rpy="0 0 ${pi}" xyz="0 0 0" />
-        <parent link="tool0" />
-        <child link="onrobot_eyes_base_link" />
-        <axis xyz="0 0 0" />
+        <origin rpy="0 0 ${pi}" xyz="0 0 0"/>
+        <parent link="tool0"/>
+        <child link="onrobot_eyes_base_link"/>
+        <axis xyz="0 0 0"/>
     </joint>
     <joint name="quick_changer_joint" type="fixed">
-        <origin rpy="0 0 ${pi/2}" xyz="0 0 0" />
-        <parent link="onrobot_eyes_tool_link" />
-        <child link="onrobot_quick_changer_base_link" />
-        <axis xyz="0 0 0" />
+        <origin rpy="0 0 ${pi/2}" xyz="0 0 0"/>
+        <parent link="onrobot_eyes_tool_link"/>
+        <child link="onrobot_quick_changer_base_link"/>
+        <axis xyz="0 0 0"/>
     </joint>
 </robot>
