Commit message: updated description file

File: workspace/src/par_pkg/urdf/ur_assembly_macro.xacro (robot description, xacro)
@@ -10,26 +10,61 @@
         name="ur_assembly"
         params="
-        parent
-        ur_type
-        joint_limits_parameters_file
-        kinematics_parameters_file
-        physical_parameters_file
-        visual_parameters_file
         low_poly:='true'
         gripper:='true'
         mounting_angle:=0
         camera_angle:=0
-    ">
-        <link name="mount_plate_link">
+        name
+    tf_prefix
+    parent
+    *origin
+    joint_limits_parameters_file
+    kinematics_parameters_file
+    physical_parameters_file
+    visual_parameters_file
+    generate_ros2_control_tag:=true
+    transmission_hw_interface:=hardware_interface/PositionJointInterface
+    safety_limits:=false
+    safety_pos_margin:=0.15
+    safety_k_position:=20
+    use_fake_hardware:=false
+    fake_sensor_commands:=false
+    sim_gazebo:=false
+    sim_ignition:=false
+    headless_mode:=false
+    initial_positions:=${dict(shoulder_pan_joint=0.0,shoulder_lift_joint=-1.57,elbow_joint=0.0,wrist_1_joint=-1.57,wrist_2_joint=0.0,wrist_3_joint=0.0)}
+    use_tool_communication:=false
+    tool_voltage:=0
+    tool_parity:=0
+    tool_baud_rate:=115200
+    tool_stop_bits:=1
+    tool_rx_idle_chars:=1.5
+    tool_tx_idle_chars:=3.5
+    tool_device_name:=/tmp/ttyUR
+    tool_tcp_port:=54321
+    robot_ip:=0.0.0.0
+    script_filename:=to_be_filled_by_ur_robot_driver
+    output_recipe_filename:=to_be_filled_by_ur_robot_driver
+    input_recipe_filename:=to_be_filled_by_ur_robot_driver
+    reverse_port:=50001
+    script_sender_port:=50002
+    reverse_ip:=0.0.0.0
+    script_command_port:=50004
+    trajectory_port:=50003
+    non_blocking_read:=true
+    keep_alive_count:=2"
+    >
+        <link name="
+    mount_plate_link">
             <visual>
-                <origin xyz="0 0 -${mount_plate_depth/2}" />
+                <origin xyz="
+    0 0 -${mount_plate_depth/ 2}" />
                 <geometry>
-                    <mesh filename="package://par_pkg/meshes/visual/base_plate.dae" />
+                    <mesh filename=" package:// par_pkg/ meshes/ visual/ base_plate.dae" />
                 </geometry>
             </visual>
             <collision>
-                <origin xyz="0 0 -${mount_plate_depth/2}" />
+                <origin xyz=" 0 0 -${mount_plate_depth/ 2}" />
                 <geometry>
-                    <box size="${mount_plate_size} ${mount_plate_size} ${mount_plate_depth}" />
+                    <box size=" ${mount_plate_size} ${mount_plate_size} ${mount_plate_depth}" />
                 </geometry>
             </collision>
@@ -37,10 +72,38 @@
         <xacro:ur_robot
             name="${ur_type}"
-            tf_prefix=""
             parent="mount_plate_link"
+            tf_prefix="${tf_prefix}"
             joint_limits_parameters_file="${joint_limits_parameters_file}"
             kinematics_parameters_file="${kinematics_parameters_file}"
             physical_parameters_file="${physical_parameters_file}"
             visual_parameters_file="${visual_parameters_file}"
+            transmission_hw_interface="${transmission_hw_interface}"
+            safety_limits="${safety_limits}"
+            safety_pos_margin="${safety_pos_margin}"
+            safety_k_position="${safety_k_position}"
+            use_fake_hardware="${use_fake_hardware}"
+            fake_sensor_commands="${fake_sensor_commands}"
+            sim_gazebo="${sim_gazebo}"
+            sim_ignition="${sim_ignition}"
+            headless_mode="${headless_mode}"
+            initial_positions="${xacro.load_yaml(initial_positions_file)}"
+            use_tool_communication="${use_tool_communication}"
+            tool_voltage="${tool_voltage}"
+            tool_parity="${tool_parity}"
+            tool_baud_rate="${tool_baud_rate}"
+            tool_stop_bits="${tool_stop_bits}"
+            tool_rx_idle_chars="${tool_rx_idle_chars}"
+            tool_tx_idle_chars="${tool_tx_idle_chars}"
+            tool_device_name="${tool_device_name}"
+            tool_tcp_port="${tool_tcp_port}"
+            robot_ip="${robot_ip}"
+            script_filename="${script_filename}"
+            output_recipe_filename="${output_recipe_filename}"
+            input_recipe_filename="${input_recipe_filename}"
+            reverse_ip="${reverse_ip}"
+            script_command_port="${script_command_port}"
+            reverse_port="${reverse_port}"
+            script_sender_port="${script_sender_port}"
+            trajectory_port="${trajectory_port}"
         >
             <origin xyz="0 0 0" rpy="0 0 0" />

File: workspace/ur.urdf.xacro (robot description, xacro)
@@ -1,8 +1,5 @@
 <?xml version="1.0"?>
-<robot xmlns:xacro="http://www.ros.org/wiki/xacro" name="ur5e">
-    <!-- There is currently no way to change this, we will need a custom launch file for the ur
-    drivers -->
-    <xacro:arg name="gripper" default="true" />
-    <!-- robot name parameter -->
+<robot xmlns:xacro="http://wiki.ros.org/xacro" name="$(arg name)">
+   <!-- robot name parameter -->
    <xacro:arg name="name" default="ur"/>
    <!-- import main macro -->
@@ -52,45 +49,66 @@
    <!-- convert to property to use substitution in function -->
    <xacro:property name="initial_positions_file" default="$(arg initial_positions_file)"/>
-    <xacro:include filename="$(find par_pkg)/urdf/ur_assembly_macro.xacro" />
-    <link name="world" />
-    <xacro:ur_assembly
-        parent="world"
-        ur_type="$(arg ur_type)"
-        gripper="$(arg gripper)"
-        name="$(arg name)"
-        tf_prefix="$(arg tf_prefix)"
-        joint_limits_parameters_file="$(arg joint_limit_params)"
-        kinematics_parameters_file="$(arg kinematics_params)"
-        physical_parameters_file="$(arg physical_params)"
-        visual_parameters_file="$(arg visual_params)"
-        transmission_hw_interface="$(arg transmission_hw_interface)"
-        safety_limits="$(arg safety_limits)"
-        safety_pos_margin="$(arg safety_pos_margin)"
-        safety_k_position="$(arg safety_k_position)"
-        use_fake_hardware="$(arg use_fake_hardware)"
-        fake_sensor_commands="$(arg fake_sensor_commands)"
-        sim_gazebo="$(arg sim_gazebo)"
-        sim_ignition="$(arg sim_ignition)"
-        headless_mode="$(arg headless_mode)"
-        initial_positions="${xacro.load_yaml(initial_positions_file)}"
-        use_tool_communication="$(arg use_tool_communication)"
-        tool_voltage="$(arg tool_voltage)"
-        tool_parity="$(arg tool_parity)"
-        tool_baud_rate="$(arg tool_baud_rate)"
-        tool_stop_bits="$(arg tool_stop_bits)"
-        tool_rx_idle_chars="$(arg tool_rx_idle_chars)"
-        tool_tx_idle_chars="$(arg tool_tx_idle_chars)"
-        tool_device_name="$(arg tool_device_name)"
-        tool_tcp_port="$(arg tool_tcp_port)"
-        robot_ip="$(arg robot_ip)"
-        script_filename="$(arg script_filename)"
-        output_recipe_filename="$(arg output_recipe_filename)"
-        input_recipe_filename="$(arg input_recipe_filename)"
-        reverse_ip="$(arg reverse_ip)"
-        script_command_port="$(arg script_command_port)"
-        reverse_port="$(arg reverse_port)"
-        script_sender_port="$(arg script_sender_port)"
-        trajectory_port="$(arg trajectory_port)"
-    >
-    </xacro:ur_assembly>
+   <!-- create link fixed to the "world" -->
+   <link name="world" />
+   <!-- arm -->
+   <xacro:ur_robot
+     name="$(arg name)"
+     tf_prefix="$(arg tf_prefix)"
+     parent="world"
+     joint_limits_parameters_file="$(arg joint_limit_params)"
+     kinematics_parameters_file="$(arg kinematics_params)"
+     physical_parameters_file="$(arg physical_params)"
+     visual_parameters_file="$(arg visual_params)"
+     transmission_hw_interface="$(arg transmission_hw_interface)"
+     safety_limits="$(arg safety_limits)"
+     safety_pos_margin="$(arg safety_pos_margin)"
+     safety_k_position="$(arg safety_k_position)"
+     use_fake_hardware="$(arg use_fake_hardware)"
+     fake_sensor_commands="$(arg fake_sensor_commands)"
+     sim_gazebo="$(arg sim_gazebo)"
+     sim_ignition="$(arg sim_ignition)"
+     headless_mode="$(arg headless_mode)"
+     initial_positions="${xacro.load_yaml(initial_positions_file)}"
+     use_tool_communication="$(arg use_tool_communication)"
+     tool_voltage="$(arg tool_voltage)"
+     tool_parity="$(arg tool_parity)"
+     tool_baud_rate="$(arg tool_baud_rate)"
+     tool_stop_bits="$(arg tool_stop_bits)"
+     tool_rx_idle_chars="$(arg tool_rx_idle_chars)"
+     tool_tx_idle_chars="$(arg tool_tx_idle_chars)"
+     tool_device_name="$(arg tool_device_name)"
+     tool_tcp_port="$(arg tool_tcp_port)"
+     robot_ip="$(arg robot_ip)"
+     script_filename="$(arg script_filename)"
+     output_recipe_filename="$(arg output_recipe_filename)"
+     input_recipe_filename="$(arg input_recipe_filename)"
+     reverse_ip="$(arg reverse_ip)"
+     script_command_port="$(arg script_command_port)"
+     reverse_port="$(arg reverse_port)"
+     script_sender_port="$(arg script_sender_port)"
+     trajectory_port="$(arg trajectory_port)"
+     >
+     <origin xyz="0 0 0" rpy="0 0 0" />          <!-- position robot in the world -->
+   </xacro:ur_robot>
+   <xacro:if value="$(arg sim_gazebo)">
+    <!-- Gazebo plugins -->
+    <gazebo reference="world">
+    </gazebo>
+    <gazebo>
+      <plugin filename="libgazebo_ros2_control.so" name="gazebo_ros2_control">
+        <parameters>$(arg simulation_controllers)</parameters>
+      </plugin>
+    </gazebo>
+  </xacro:if>
+  <xacro:if value="$(arg sim_ignition)">
+    <!-- Gazebo plugins -->
+    <gazebo reference="world">
+    </gazebo>
+    <gazebo>
+      <plugin filename="libign_ros2_control-system.so" name="ign_ros2_control::IgnitionROS2ControlPlugin">
+        <parameters>$(arg simulation_controllers)</parameters>
+        <controller_manager_node_name>$(arg tf_prefix)controller_manager</controller_manager_node_name>
+      </plugin>
+    </gazebo>
+  </xacro:if>
 </robot>

Commit message: tried to fix weird missing mount plate bug

File: workspace/src/par_pkg/urdf/ur_assembly_macro.xacro (robot description, xacro)
@@ -16,55 +16,53 @@
         name
         ur_type
-    tf_prefix
-    parent
-    joint_limits_parameters_file
-    kinematics_parameters_file
-    physical_parameters_file
-    visual_parameters_file
-    generate_ros2_control_tag:=true
-    transmission_hw_interface:=hardware_interface/PositionJointInterface
-    safety_limits:=false
-    safety_pos_margin:=0.15
-    safety_k_position:=20
-    use_fake_hardware:=false
-    fake_sensor_commands:=false
-    sim_gazebo:=false
-    sim_ignition:=false
-    headless_mode:=false
-    initial_positions:=${dict(shoulder_pan_joint=0.0,shoulder_lift_joint=-1.57,elbow_joint=0.0,wrist_1_joint=-1.57,wrist_2_joint=0.0,wrist_3_joint=0.0)}
-    use_tool_communication:=false
-    tool_voltage:=0
-    tool_parity:=0
-    tool_baud_rate:=115200
-    tool_stop_bits:=1
-    tool_rx_idle_chars:=1.5
-    tool_tx_idle_chars:=3.5
-    tool_device_name:=/tmp/ttyUR
-    tool_tcp_port:=54321
-    robot_ip:=0.0.0.0
-    script_filename:=to_be_filled_by_ur_robot_driver
-    output_recipe_filename:=to_be_filled_by_ur_robot_driver
-    input_recipe_filename:=to_be_filled_by_ur_robot_driver
-    reverse_port:=50001
-    script_sender_port:=50002
-    reverse_ip:=0.0.0.0
-    script_command_port:=50004
-    trajectory_port:=50003
-    non_blocking_read:=true
-    keep_alive_count:=2"
+        tf_prefix
+        parent
+        joint_limits_parameters_file
+        kinematics_parameters_file
+        physical_parameters_file
+        visual_parameters_file
+        generate_ros2_control_tag:=true
+        transmission_hw_interface:=hardware_interface/PositionJointInterface
+        safety_limits:=false
+        safety_pos_margin:=0.15
+        safety_k_position:=20
+        use_fake_hardware:=false
+        fake_sensor_commands:=false
+        sim_gazebo:=false
+        sim_ignition:=false
+        headless_mode:=false
+        initial_positions:=${dict(shoulder_pan_joint=0.0,shoulder_lift_joint=-1.57,elbow_joint=0.0,wrist_1_joint=-1.57,wrist_2_joint=0.0,wrist_3_joint=0.0)}
+        use_tool_communication:=false
+        tool_voltage:=0
+        tool_parity:=0
+        tool_baud_rate:=115200
+        tool_stop_bits:=1
+        tool_rx_idle_chars:=1.5
+        tool_tx_idle_chars:=3.5
+        tool_device_name:=/tmp/ttyUR
+        tool_tcp_port:=54321
+        robot_ip:=0.0.0.0
+        script_filename:=to_be_filled_by_ur_robot_driver
+        output_recipe_filename:=to_be_filled_by_ur_robot_driver
+        input_recipe_filename:=to_be_filled_by_ur_robot_driver
+        reverse_port:=50001
+        script_sender_port:=50002
+        reverse_ip:=0.0.0.0
+        script_command_port:=50004
+        trajectory_port:=50003
+        non_blocking_read:=true
+        keep_alive_count:=2"
     >
-        <link name="
-    mount_plate_link">
+        <link name="mount_plate_link">
             <visual>
-                <origin xyz="
-    0 0 -${mount_plate_depth/ 2}" />
+                <origin xyz="0 0 -${mount_plate_depth/ 2}" />
                 <geometry>
-                    <mesh filename=" package:// par_pkg/ meshes/ visual/ base_plate.dae" />
+                    <mesh filename="package://par_pkg/meshes/visual/base_plate.dae" />
                 </geometry>
             </visual>
             <collision>
-                <origin xyz=" 0 0 -${mount_plate_depth/ 2}" />
+                <origin xyz="0 0 -${mount_plate_depth/ 2}" />
                 <geometry>
-                    <box size=" ${mount_plate_size} ${mount_plate_size} ${mount_plate_depth}" />
+                    <box size="${mount_plate_size} ${mount_plate_size} ${mount_plate_depth}" />
                 </geometry>
             </collision>

Commit message: Mount plate link goes to world now

File: workspace/src/par_pkg/urdf/ur_assembly_macro.xacro (robot description, xacro)
@@ -122,5 +122,5 @@
         <joint name="mount_plate_joint" type="fixed">
             <origin xyz="0 0 ${mount_plate_depth}" rpy="0 0 ${mounting_angle}" />
-            <parent link="world" />
+            <parent link="${parent}" />
             <child link="mount_plate_link" />
         </joint>
