Commit message: Set up the new xacro files

File: workspace/src/par_pkg/urdf/onrobot_rg2.xacro (robot description, xacro)
@@ -1,8 +1,21 @@
 <?xml version="1.0"?>
-<robot name="onrobot_rg2_gripper">
+<robot xmlns:xacro="http://www.ros.org/wiki/xacro" name="onrobot_rg2_gripper">
+    <xacro:macro
+    name="onrobot_rg2_gripper"
+    params="
+        parent
+        low_poly:=true
+    "
+    >
+    <xacro:if value="${low_poly}">
+        <xacro:property name="poly" value="_low_poly"/>
+    </xacro:if>
+    <xacro:if value="${not low_poly}">
+        <xacro:property name="poly" value=""/>
+    </xacro:if>
     <link name="onrobot_rg2_base_link">
         <visual>
             <geometry>
-                <mesh filename="package://par_pkg/meshes/visual/rg2_base_link_v2.dae" />
+                <mesh filename="package://par_pkg/meshes/visual/rg2_base_link${poly}.dae" />
             </geometry>
         </visual>
@@ -16,5 +29,5 @@
         <visual>
             <geometry>
-                <mesh filename="package://par_pkg/meshes/visual/rg2_outer_knuckle_v2.dae" />
+                <mesh filename="package://par_pkg/meshes/visual/rg2_outer_knuckle${poly}.dae" />
             </geometry>
         </visual>
@@ -28,5 +41,5 @@
         <visual>
             <geometry>
-                <mesh filename="package://par_pkg/meshes/visual/rg2_inner_knuckle_v2.dae" />
+                <mesh filename="package://par_pkg/meshes/visual/rg2_inner_knuckle${poly}.dae" />
             </geometry>
         </visual>
@@ -40,5 +53,5 @@
         <visual>
             <geometry>
-                <mesh filename="package://par_pkg/meshes/visual/rg2_finger_v2.dae" />
+                <mesh filename="package://par_pkg/meshes/visual/rg2_finger${poly}.dae" />
             </geometry>
         </visual>
@@ -52,5 +65,5 @@
         <visual>
             <geometry>
-                <mesh filename="package://par_pkg/meshes/visual/rg2_outer_knuckle_v2.dae" />
+                <mesh filename="package://par_pkg/meshes/visual/rg2_outer_knuckle${poly}.dae" />
             </geometry>
         </visual>
@@ -64,5 +77,5 @@
         <visual>
             <geometry>
-                <mesh filename="package://par_pkg/meshes/visual/rg2_inner_knuckle_v2.dae" />
+                <mesh filename="package://par_pkg/meshes/visual/rg2_inner_knuckle${poly}.dae" />
             </geometry>
         </visual>
@@ -76,5 +89,5 @@
         <visual>
             <geometry>
-                <mesh filename="package://par_pkg/meshes/visual/rg2_finger_v2.dae" />
+                <mesh filename="package://par_pkg/meshes/visual/rg2_finger${poly}.dae" />
             </geometry>
         </visual>
@@ -86,4 +99,8 @@
     </link>
     <!-- <link name="grip_point"/> -->
+    <joint name="rg2_parent_joint" type="fixed">
+        <parent link="${parent}"/>
+        <child link="onrobot_rg2_base_link"/>
+    </joint>
     <joint name="finger_joint" type="revolute">
         <origin rpy="0 0 1.57079632679" xyz="-0.01 -0.01705 0.1207" />
@@ -142,3 +159,4 @@
         </actuator>
       </transmission>
+    </xacro:macro>
 </robot>

File: workspace/src/par_pkg/urdf/ur_assembly.urdf.xacro (robot description, xacro)
@@ -1,4 +1,6 @@
 <?xml version="1.0"?>
 <robot xmlns:xacro="http://www.ros.org/wiki/xacro" name="ur5e">
+    <!-- There is currently no way to change this, we will need a custom launch file for the ur drivers -->
+    <xacro:arg name="gripper" default="true"/>
     <xacro:arg name="ur_type" default="ur5e"/>
     <xacro:arg name="joint_limit_params"
@@ -19,4 +21,5 @@
         physical_parameters_file="$(arg physical_params)"
         visual_parameters_file="$(arg visual_params)"
+        gripper="$(arg gripper)"
     >
     </xacro:ur_assembly>

File: workspace/src/par_pkg/urdf/ur_assembly_macro.xacro (robot description, xacro)
@@ -4,6 +4,6 @@
     <xacro:include filename="$(find par_pkg)/urdf/onrobot_eyes.xacro" />
     <xacro:include filename="$(find par_pkg)/urdf/onrobot_quick_changer.xacro" />
-    <xacro:include filename="$(find par_pkg)/urdf/onrobot_rg2_gripper.urdf"/>
-    <xacro:property name="mount_plate_size" value="0.2" />
+    <xacro:include filename="$(find par_pkg)/urdf/onrobot_rg2.xacro" />
+    <xacro:property name="mount_plate_size" value="0.194" />
     <xacro:property name="mount_plate_depth" value="0.0127" />
     <xacro:macro
@@ -21,13 +21,9 @@
         camera_angle:=0
     ">
-        <joint name="gripper" type="fixed">
-            <parent link="onrobot_quick_changer_tool_link"/>
-            <child link="onrobot_rg2_base_link"/>
-        </joint>
         <link name="mount_plate_link">
             <visual>
                 <origin xyz="0 0 -${mount_plate_depth/2}" />
                 <geometry>
-                    <box size="${mount_plate_size} ${mount_plate_size} ${mount_plate_depth}" />
+                    <mesh filename="package://par_pkg/meshes/visual/base_plate.dae" />
                 </geometry>
             </visual>
@@ -56,7 +52,11 @@
         />
         <xacro:onrobot_quick_changer
-            parent="onrobot_eyes_base_link"
+            parent="onrobot_eyes_tool_link"
             low_poly="${low_poly}"
         />
+        <xacro:if value="${gripper}">
+            <xacro:onrobot_rg2_gripper parent="onrobot_quick_changer_tool_link"
+                low_poly="${low_poly}" />
+        </xacro:if>
         <joint name="mount_plate_joint" type="fixed">
             <origin xyz="0 0 ${mount_plate_depth}" rpy="0 0 ${mounting_angle}" />

Commit message: gripper shouldnt go through table anymore

File: workspace/src/par_pkg/urdf/onrobot_rg2.xacro (robot description, xacro)
@@ -154,5 +154,5 @@
         <link name="end_effector_link" />
         <joint name="end_effector_joint" type="fixed">
-            <origin xyz="0 0 0.2246"/>
+            <origin xyz="0 0 0.2311"/>
             <parent link="onrobot_rg2_base_link" />
             <child link="end_effector_link" />

Commit message: Updated angle max

File: workspace/src/par_pkg/urdf/onrobot_rg2.xacro (robot description, xacro)
@@ -8,4 +8,5 @@
     "
     >
+        <xacro:property name="angle_max" value="3.2"/>
         <xacro:property name="knuckle_yaw" value="1.57079632679"/>
         <xacro:property name="knuckle_x_offset" value="0.01"/>
@@ -100,5 +101,4 @@
             </collision>
         </link>
-        <!-- <link name="grip_point"/> -->
         <joint name="rg2_parent_joint" type="fixed">
             <parent link="${parent}" />
@@ -110,5 +110,5 @@
             <child link="left_outer_knuckle" />
             <axis xyz="0 1 0" />
-            <limit effort="1000" lower="1.87361095202" upper="3.18697121414" velocity="1.0" />
+            <limit effort="1000" lower="1.87361095202" upper="${angle_max}" velocity="1.0" />
         </joint>
         <joint name="right_outer_knuckle_joint" type="revolute">
@@ -117,5 +117,5 @@
             <child link="right_outer_knuckle" />
             <axis xyz="0 1 0" />
-            <limit effort="1000" lower="1.87361095202" upper="3.18697121414" velocity="1.0" />
+            <limit effort="1000" lower="1.87361095202" upper="${angle_max}" velocity="1.0" />
             <mimic joint="finger_joint" multiplier="1" offset="0" />
         </joint>
@@ -125,5 +125,5 @@
             <child link="left_inner_knuckle" />
             <axis xyz="0 1 0" />
-            <limit effort="1000" lower="1.87361095202" upper="3.18697121414" velocity="1.0" />
+            <limit effort="1000" lower="1.87361095202" upper="${angle_max}" velocity="1.0" />
             <mimic joint="finger_joint" multiplier="1" offset="0" />
         </joint>
@@ -133,5 +133,5 @@
             <child link="right_inner_knuckle" />
             <axis xyz="0 1 0" />
-            <limit effort="1000" lower="1.87361095202" upper="3.18697121414" velocity="1.0" />
+            <limit effort="1000" lower="1.87361095202" upper="${angle_max}" velocity="1.0" />
             <mimic joint="finger_joint" multiplier="1" offset="0" />
         </joint>
@@ -141,5 +141,5 @@
             <child link="left_finger" />
             <axis xyz="0 0 -1" />
-            <limit effort="1000" lower="1.87361095202" upper="3.18697121414" velocity="1.0" />
+            <limit effort="1000" lower="1.87361095202" upper="${angle_max}" velocity="1.0" />
             <mimic joint="finger_joint" multiplier="-1" offset="0" />
         </joint>
@@ -149,5 +149,5 @@
             <child link="right_finger" />
             <axis xyz="0 0 1" />
-            <limit effort="1000" lower="1.87361095202" upper="3.18697121414" velocity="1.0" />
+            <limit effort="1000" lower="1.87361095202" upper="${angle_max}" velocity="1.0" />
             <mimic joint="finger_joint" multiplier="1" offset="0" />
         </joint>

Commit message: Calbirating angle max

File: workspace/src/par_pkg/urdf/onrobot_rg2.xacro (robot description, xacro)
@@ -8,5 +8,5 @@
     "
     >
-        <xacro:property name="angle_max" value="3.2"/>
+        <xacro:property name="angle_max" value="3.3"/>
         <xacro:property name="knuckle_yaw" value="1.57079632679"/>
         <xacro:property name="knuckle_x_offset" value="0.01"/>

Commit message: Actually updating the correct value now

File: workspace/src/par_pkg/urdf/onrobot_rg2.xacro (robot description, xacro)
@@ -8,5 +8,6 @@
     "
     >
-        <xacro:property name="angle_max" value="3.3"/>
+        <xacro:property name="angle_max" value="3.18697121414"/>
+        <xacro:property name="angle_min" value="1.8"/>
         <xacro:property name="knuckle_yaw" value="1.57079632679"/>
         <xacro:property name="knuckle_x_offset" value="0.01"/>
@@ -110,5 +111,5 @@
             <child link="left_outer_knuckle" />
             <axis xyz="0 1 0" />
-            <limit effort="1000" lower="1.87361095202" upper="${angle_max}" velocity="1.0" />
+            <limit effort="1000" lower="${angle_min}" upper="${angle_max}" velocity="1.0" />
         </joint>
         <joint name="right_outer_knuckle_joint" type="revolute">
@@ -117,5 +118,5 @@
             <child link="right_outer_knuckle" />
             <axis xyz="0 1 0" />
-            <limit effort="1000" lower="1.87361095202" upper="${angle_max}" velocity="1.0" />
+            <limit effort="1000" lower="${angle_min}" upper="${angle_max}" velocity="1.0" />
             <mimic joint="finger_joint" multiplier="1" offset="0" />
         </joint>
@@ -125,5 +126,5 @@
             <child link="left_inner_knuckle" />
             <axis xyz="0 1 0" />
-            <limit effort="1000" lower="1.87361095202" upper="${angle_max}" velocity="1.0" />
+            <limit effort="1000" lower="${angle_min}" upper="${angle_max}" velocity="1.0" />
             <mimic joint="finger_joint" multiplier="1" offset="0" />
         </joint>
@@ -133,5 +134,5 @@
             <child link="right_inner_knuckle" />
             <axis xyz="0 1 0" />
-            <limit effort="1000" lower="1.87361095202" upper="${angle_max}" velocity="1.0" />
+            <limit effort="1000" lower="${angle_min}" upper="${angle_max}" velocity="1.0" />
             <mimic joint="finger_joint" multiplier="1" offset="0" />
         </joint>
@@ -141,5 +142,5 @@
             <child link="left_finger" />
             <axis xyz="0 0 -1" />
-            <limit effort="1000" lower="1.87361095202" upper="${angle_max}" velocity="1.0" />
+            <limit effort="1000" lower="${angle_min}" upper="${angle_max}" velocity="1.0" />
             <mimic joint="finger_joint" multiplier="-1" offset="0" />
         </joint>
@@ -149,5 +150,5 @@
             <child link="right_finger" />
             <axis xyz="0 0 1" />
-            <limit effort="1000" lower="1.87361095202" upper="${angle_max}" velocity="1.0" />
+            <limit effort="1000" lower="${angle_min}" upper="${angle_max}" velocity="1.0" />
             <mimic joint="finger_joint" multiplier="1" offset="0" />
         </joint>

Commit message: updated angle again

File: workspace/src/par_pkg/urdf/onrobot_rg2.xacro (robot description, xacro)
@@ -9,5 +9,5 @@
     >
         <xacro:property name="angle_max" value="3.18697121414"/>
-        <xacro:property name="angle_min" value="1.8"/>
+        <xacro:property name="angle_min" value="1.7"/>
         <xacro:property name="knuckle_yaw" value="1.57079632679"/>
         <xacro:property name="knuckle_x_offset" value="0.01"/>

Commit message: Overshot by a lot for testing

File: workspace/src/par_pkg/urdf/onrobot_rg2.xacro (robot description, xacro)
@@ -9,5 +9,5 @@
     >
         <xacro:property name="angle_max" value="3.18697121414"/>
-        <xacro:property name="angle_min" value="1.7"/>
+        <xacro:property name="angle_min" value="1.5"/>
         <xacro:property name="knuckle_yaw" value="1.57079632679"/>
         <xacro:property name="knuckle_x_offset" value="0.01"/>

Commit message: Reversed everything

File: workspace/src/par_pkg/urdf/onrobot_rg2.xacro (robot description, xacro)
@@ -9,5 +9,5 @@
     >
         <xacro:property name="angle_max" value="3.18697121414"/>
-        <xacro:property name="angle_min" value="1.5"/>
+        <xacro:property name="angle_min" value="1.87361095202"/>
         <xacro:property name="knuckle_yaw" value="1.57079632679"/>
         <xacro:property name="knuckle_x_offset" value="0.01"/>
