Commit message: replaced world with map

File: workspace/src/par_pkg/urdf/ur_assembly.urdf.xacro (robot description, xacro)
@@ -53,7 +53,7 @@
    <xacro:property name="initial_positions_file" default="$(arg initial_positions_file)"/>
     <xacro:include filename="$(find par_pkg)/urdf/ur_assembly_macro.xacro" />
-    <link name="world" />
+    <link name="map" />
     <xacro:ur_assembly
-        parent="world"
+        parent="map"
         ur_type="$(arg ur_type)"
         gripper="$(arg gripper)"

Commit message: Added map frame as its own thing

File: workspace/src/par_pkg/urdf/ur_assembly.urdf.xacro (robot description, xacro)
@@ -53,7 +53,12 @@
    <xacro:property name="initial_positions_file" default="$(arg initial_positions_file)"/>
     <xacro:include filename="$(find par_pkg)/urdf/ur_assembly_macro.xacro" />
+    <link name="world"/>
     <link name="map" />
+    <joint name="map_joint" type="fixed">
+      <parent link="world"/>
+      <child name="map"/>
+    </joint>
     <xacro:ur_assembly
-        parent="map"
+        parent="world"
         ur_type="$(arg ur_type)"
         gripper="$(arg gripper)"

Commit message: Fixed typo in map frame

File: workspace/src/par_pkg/urdf/ur_assembly.urdf.xacro (robot description, xacro)
@@ -57,5 +57,5 @@
     <joint name="map_joint" type="fixed">
       <parent link="world"/>
-      <child name="map"/>
+      <child link="map"/>
     </joint>
     <xacro:ur_assembly
