Commit message: Added end effector joint

File: workspace/src/par_pkg/urdf/onrobot_eyes.xacro (robot description, xacro)
@@ -2,4 +2,7 @@
 <robot xmlns:xacro="http://www.ros.org/wiki/xacro" name="onrobot_eyes">
     <xacro:include filename="$(find realsense2_description)/urdf/_d415.urdf.xacro" />
+    <xacro:property name="d415_cam_depth_py" value="0.020"/>
+    <xacro:property name="d415_cam_depth_pz" value="${d415_cam_height/2}"/>
+    <xacro:property name="d415_cam_height" value="0.023"/>
     <xacro:macro name="onrobot_eyes"
         params="
@@ -16,5 +19,5 @@
             industrial_calibration seems like a good package for doing this.
         -->
-            <origin xyz="-0.01091 0.105055 0.019792" rpy="-${pi/2} -${pi/2} 0" />
+            <origin xyz="0 ${0.10485-d415_cam_depth_py/2} 0.019792" rpy="-${pi/2} -${pi/2} 0" />
         </xacro:sensor_d415>
         <link name="onrobot_eyes_base_link"/>
@@ -25,7 +28,7 @@
                         <mesh filename="package://par_pkg/meshes/visual/onrobot_eyes_low_poly.dae" />
                     </xacro:if>
-                    <xacro:if value="${not low_poly}">
+                    <xacro:unless value="${low_poly}">
                         <mesh filename="package://par_pkg/meshes/visual/onrobot_eyes.dae" />
-                    </xacro:if>
+                    </xacro:unless>
                 </geometry>
             </visual>

File: workspace/src/par_pkg/urdf/onrobot_quick_changer.xacro (robot description, xacro)
@@ -13,7 +13,7 @@
                         <mesh filename="package://par_pkg/meshes/visual/quick_changer_low_poly.dae" />
                     </xacro:if>
-                    <xacro:if value="${not low_poly}">
+                    <xacro:unless value="${low_poly}">
                         <mesh filename="package://par_pkg/meshes/visual/quick_changer.dae" />
-                    </xacro:if>
+                    </xacro:unless>
                 </geometry>
             </visual>

File: workspace/src/par_pkg/urdf/onrobot_rg2.xacro (robot description, xacro)
@@ -2,161 +2,169 @@
 <robot xmlns:xacro="http://www.ros.org/wiki/xacro" name="onrobot_rg2_gripper">
     <xacro:macro
-    name="onrobot_rg2_gripper"
-    params="
+        name="onrobot_rg2_gripper"
+        params="
         parent
         low_poly:=true
     "
     >
-    <xacro:if value="${low_poly}">
-        <xacro:property name="poly" value="_low_poly"/>
-    </xacro:if>
-    <xacro:if value="${not low_poly}">
-        <xacro:property name="poly" value=""/>
-    </xacro:if>
-    <link name="onrobot_rg2_base_link">
-        <visual>
-            <geometry>
-                <mesh filename="package://par_pkg/meshes/visual/rg2_base_link${poly}.dae" />
-            </geometry>
-        </visual>
-        <collision>
-            <geometry>
-                <mesh filename="package://par_pkg/meshes/collision/rg2_base_link.stl" />
-            </geometry>
-        </collision>
-    </link>
-    <link name="left_outer_knuckle">
-        <visual>
-            <geometry>
-                <mesh filename="package://par_pkg/meshes/visual/rg2_outer_knuckle${poly}.dae" />
-            </geometry>
-        </visual>
-        <collision>
-            <geometry>
-                <mesh filename="package://par_pkg/meshes/collision/rg2_outer_knuckle.stl" />
-            </geometry>
-        </collision>
-    </link>
-    <link name="left_inner_knuckle">
-        <visual>
-            <geometry>
-                <mesh filename="package://par_pkg/meshes/visual/rg2_inner_knuckle${poly}.dae" />
-            </geometry>
-        </visual>
-        <collision>
-            <geometry>
-                <mesh filename="package://par_pkg/meshes/collision/rg2_inner_knuckle.stl" />
-            </geometry>
-        </collision>
-    </link>
-    <link name="left_finger">
-        <visual>
-            <geometry>
-                <mesh filename="package://par_pkg/meshes/visual/rg2_finger${poly}.dae" />
-            </geometry>
-        </visual>
-        <collision>
-            <geometry>
-                <mesh filename="package://par_pkg/meshes/collision/rg2_finger.stl" />
-            </geometry>
-        </collision>
-    </link>
-    <link name="right_outer_knuckle">
-        <visual>
-            <geometry>
-                <mesh filename="package://par_pkg/meshes/visual/rg2_outer_knuckle${poly}.dae" />
-            </geometry>
-        </visual>
-        <collision>
-            <geometry>
-                <mesh filename="package://par_pkg/meshes/collision/rg2_outer_knuckle.stl" />
-            </geometry>
-        </collision>
-    </link>
-    <link name="right_inner_knuckle">
-        <visual>
-            <geometry>
-                <mesh filename="package://par_pkg/meshes/visual/rg2_inner_knuckle${poly}.dae" />
-            </geometry>
-        </visual>
-        <collision>
-            <geometry>
-                <mesh filename="package://par_pkg/meshes/collision/rg2_inner_knuckle.stl" />
-            </geometry>
-        </collision>
-    </link>
-    <link name="right_finger">
-        <visual>
-            <geometry>
-                <mesh filename="package://par_pkg/meshes/visual/rg2_finger${poly}.dae" />
-            </geometry>
-        </visual>
-        <collision>
-            <geometry>
-                <mesh filename="package://par_pkg/meshes/collision/rg2_finger.stl" />
-            </geometry>
-        </collision>
-    </link>
-    <!-- <link name="grip_point"/> -->
-    <joint name="rg2_parent_joint" type="fixed">
-        <parent link="${parent}"/>
-        <child link="onrobot_rg2_base_link"/>
-    </joint>
-    <joint name="finger_joint" type="revolute">
-        <origin rpy="0 0 1.57079632679" xyz="-0.01 -0.01705 0.1207" />
-        <parent link="onrobot_rg2_base_link" />
-        <child link="left_outer_knuckle" />
-        <axis xyz="0 1 0" />
-        <limit effort="1000" lower="1.87361095202" upper="3.18697121414" velocity="1.0" />
-    </joint>
-    <joint name="right_outer_knuckle_joint" type="revolute">
-        <origin rpy="0 0 -1.57079632679" xyz="0.01 0.01695 0.1207"/>
-        <parent link="onrobot_rg2_base_link"/>
-        <child link="right_outer_knuckle"/>
-        <axis xyz="0 1 0"/>
-        <limit effort="1000" lower="1.87361095202" upper="3.18697121414" velocity="1.0" />
-        <mimic joint="finger_joint" multiplier="1" offset="0"/>
-      </joint>
-      <joint name="left_inner_knuckle_joint" type="revolute">
-        <origin rpy="0 0 1.57079632679" xyz="0.01 -0.00755 0.1372"/>
-        <parent link="onrobot_rg2_base_link"/>
-        <child link="left_inner_knuckle"/>
-        <axis xyz="0 1 0"/>
-        <limit effort="1000" lower="1.87361095202" upper="3.18697121414" velocity="1.0" />
-        <mimic joint="finger_joint" multiplier="1" offset="0"/>
-      </joint>
-      <joint name="right_inner_knuckle_joint" type="revolute">
-        <origin rpy="0 0 -1.57079632679" xyz="-0.01 0.00745 0.1372"/>
-        <parent link="onrobot_rg2_base_link"/>
-        <child link="right_inner_knuckle"/>
-        <axis xyz="0 1 0"/>
-        <limit effort="1000" lower="1.87361095202" upper="3.18697121414" velocity="1.0" />
-        <mimic joint="finger_joint" multiplier="1" offset="0"/>
-      </joint>
-      <joint name="left_finger_joint" type="revolute">
-        <origin rpy="1.57079632679 -0.974896 0" xyz=" 0 -0.01 -0.055"/>
-        <parent link="left_outer_knuckle"/>
-        <child link="left_finger"/>
-        <axis xyz="0 0 -1"/>
-        <limit effort="1000" lower="1.87361095202" upper="3.18697121414" velocity="1.0" />
-        <mimic joint="finger_joint" multiplier="-1" offset="0"/>
-      </joint>
-      <joint name="right_finger_joint" type="revolute">
-        <origin rpy="1.57079632679 -0.974896 0" xyz=" 0 -0.01 -0.055"/>
-        <parent link="right_outer_knuckle"/>
-        <child link="right_finger"/>
-        <axis xyz="0 0 1"/>
-        <limit effort="1000" lower="1.87361095202" upper="3.18697121414" velocity="1.0" />
-        <mimic joint="finger_joint" multiplier="1" offset="0"/>
-      </joint>
-      <transmission name="finger_joint_trans">
-        <type>transmission_interface/SimpleTransmission</type>
-        <joint name="finger_joint">
-          <hardwareInterface>PositionJointInterface</hardwareInterface>
+        <xacro:property name="knuckle_yaw" value="1.57079632679"/>
+        <xacro:property name="knuckle_x_offset" value="0.01"/>
+        <xacro:if value="${low_poly}">
+            <xacro:property name="poly" value="_low_poly" />
+        </xacro:if>
+        <xacro:unless value="${low_poly}">
+            <xacro:property name="poly" value="" />
+        </xacro:unless>
+        <link name="onrobot_rg2_base_link">
+            <visual>
+                <geometry>
+                    <mesh filename="package://par_pkg/meshes/visual/rg2_base_link${poly}.dae" />
+                </geometry>
+            </visual>
+            <collision>
+                <geometry>
+                    <mesh filename="package://par_pkg/meshes/collision/rg2_base_link.stl" />
+                </geometry>
+            </collision>
+        </link>
+        <link name="left_outer_knuckle">
+            <visual>
+                <geometry>
+                    <mesh filename="package://par_pkg/meshes/visual/rg2_outer_knuckle${poly}.dae" />
+                </geometry>
+            </visual>
+            <collision>
+                <geometry>
+                    <mesh filename="package://par_pkg/meshes/collision/rg2_outer_knuckle.stl" />
+                </geometry>
+            </collision>
+        </link>
+        <link name="left_inner_knuckle">
+            <visual>
+                <geometry>
+                    <mesh filename="package://par_pkg/meshes/visual/rg2_inner_knuckle${poly}.dae" />
+                </geometry>
+            </visual>
+            <collision>
+                <geometry>
+                    <mesh filename="package://par_pkg/meshes/collision/rg2_inner_knuckle.stl" />
+                </geometry>
+            </collision>
+        </link>
+        <link name="left_finger">
+            <visual>
+                <geometry>
+                    <mesh filename="package://par_pkg/meshes/visual/rg2_finger${poly}.dae" />
+                </geometry>
+            </visual>
+            <collision>
+                <geometry>
+                    <mesh filename="package://par_pkg/meshes/collision/rg2_finger.stl" />
+                </geometry>
+            </collision>
+        </link>
+        <link name="right_outer_knuckle">
+            <visual>
+                <geometry>
+                    <mesh filename="package://par_pkg/meshes/visual/rg2_outer_knuckle${poly}.dae" />
+                </geometry>
+            </visual>
+            <collision>
+                <geometry>
+                    <mesh filename="package://par_pkg/meshes/collision/rg2_outer_knuckle.stl" />
+                </geometry>
+            </collision>
+        </link>
+        <link name="right_inner_knuckle">
+            <visual>
+                <geometry>
+                    <mesh filename="package://par_pkg/meshes/visual/rg2_inner_knuckle${poly}.dae" />
+                </geometry>
+            </visual>
+            <collision>
+                <geometry>
+                    <mesh filename="package://par_pkg/meshes/collision/rg2_inner_knuckle.stl" />
+                </geometry>
+            </collision>
+        </link>
+        <link name="right_finger">
+            <visual>
+                <geometry>
+                    <mesh filename="package://par_pkg/meshes/visual/rg2_finger${poly}.dae" />
+                </geometry>
+            </visual>
+            <collision>
+                <geometry>
+                    <mesh filename="package://par_pkg/meshes/collision/rg2_finger.stl" />
+                </geometry>
+            </collision>
+        </link>
+        <!-- <link name="grip_point"/> -->
+        <joint name="rg2_parent_joint" type="fixed">
+            <parent link="${parent}" />
+            <child link="onrobot_rg2_base_link" />
         </joint>
-        <actuator name="finger_joint_motor">
-          <mechanicalReduction>1</mechanicalReduction>
-        </actuator>
-      </transmission>
+        <joint name="finger_joint" type="revolute">
+            <origin rpy="0 0 ${knuckle_yaw}" xyz="${-knuckle_x_offset} -0.01705 0.1207" />
+            <parent link="onrobot_rg2_base_link" />
+            <child link="left_outer_knuckle" />
+            <axis xyz="0 1 0" />
+            <limit effort="1000" lower="1.87361095202" upper="3.18697121414" velocity="1.0" />
+        </joint>
+        <joint name="right_outer_knuckle_joint" type="revolute">
+            <origin rpy="0 0 ${-knuckle_yaw}" xyz="${knuckle_x_offset} 0.01695 0.1207" />
+            <parent link="onrobot_rg2_base_link" />
+            <child link="right_outer_knuckle" />
+            <axis xyz="0 1 0" />
+            <limit effort="1000" lower="1.87361095202" upper="3.18697121414" velocity="1.0" />
+            <mimic joint="finger_joint" multiplier="1" offset="0" />
+        </joint>
+        <joint name="left_inner_knuckle_joint" type="revolute">
+            <origin rpy="0 0 ${knuckle_yaw}" xyz="${knuckle_x_offset} -0.00755 0.1372" />
+            <parent link="onrobot_rg2_base_link" />
+            <child link="left_inner_knuckle" />
+            <axis xyz="0 1 0" />
+            <limit effort="1000" lower="1.87361095202" upper="3.18697121414" velocity="1.0" />
+            <mimic joint="finger_joint" multiplier="1" offset="0" />
+        </joint>
+        <joint name="right_inner_knuckle_joint" type="revolute">
+            <origin rpy="0 0 ${-knuckle_yaw}" xyz="${-knuckle_x_offset} 0.00745 0.1372" />
+            <parent link="onrobot_rg2_base_link" />
+            <child link="right_inner_knuckle" />
+            <axis xyz="0 1 0" />
+            <limit effort="1000" lower="1.87361095202" upper="3.18697121414" velocity="1.0" />
+            <mimic joint="finger_joint" multiplier="1" offset="0" />
+        </joint>
+        <joint name="left_finger_joint" type="revolute">
+            <origin rpy="1.57079632679 -0.974896 0" xyz=" 0 -0.01 -0.055" />
+            <parent link="left_outer_knuckle" />
+            <child link="left_finger" />
+            <axis xyz="0 0 -1" />
+            <limit effort="1000" lower="1.87361095202" upper="3.18697121414" velocity="1.0" />
+            <mimic joint="finger_joint" multiplier="-1" offset="0" />
+        </joint>
+        <joint name="right_finger_joint" type="revolute">
+            <origin rpy="1.57079632679 -0.974896 0" xyz=" 0 -0.01 -0.055" />
+            <parent link="right_outer_knuckle" />
+            <child link="right_finger" />
+            <axis xyz="0 0 1" />
+            <limit effort="1000" lower="1.87361095202" upper="3.18697121414" velocity="1.0" />
+            <mimic joint="finger_joint" multiplier="1" offset="0" />
+        </joint>
+        <link name="end_effector_link" />
+        <joint name="end_effector_joint" type="fixed">
+            <origin xyz="0 0 0.2246"/>
+            <parent link="onrobot_rg2_base_link" />
+            <child link="end_effector_link" />
+        </joint>
+        <transmission name="finger_joint_trans">
+            <type>transmission_interface/SimpleTransmission</type>
+            <joint name="finger_joint">
+                <hardwareInterface>PositionJointInterface</hardwareInterface>
+            </joint>
+            <actuator name="finger_joint_motor">
+                <mechanicalReduction>1</mechanicalReduction>
+            </actuator>
+        </transmission>
     </xacro:macro>
 </robot>

Commit message: updated transform diff

File: workspace/src/par_pkg/urdf/onrobot_eyes.xacro (robot description, xacro)
@@ -19,5 +19,5 @@
             industrial_calibration seems like a good package for doing this.
         -->
-            <origin xyz="0 ${0.10485-d415_cam_depth_py/2} 0.019792" rpy="-${pi/2} -${pi/2} 0" />
+            <origin xyz="0 ${0.10485-d415_cam_depth_py/2} ${0.019792+0.009}" rpy="-${pi/2} -${pi/2} 0" />
         </xacro:sensor_d415>
         <link name="onrobot_eyes_base_link"/>

Commit message: updated transform of links so now the depth frame z is properly aligned

File: workspace/src/par_pkg/urdf/onrobot_eyes.xacro (robot description, xacro)
@@ -15,9 +15,10 @@
             <!--
             These measurements are not 100% accurate, they're the best
-            I could get based on manually aligning it in blender.
+            I could get based on manually aligning it in blender, and
+            manual calibrations with transforms
             We need to preform camera extrinsics calibration manually to get these values.
             industrial_calibration seems like a good package for doing this.
         -->
-            <origin xyz="0 ${0.10485-d415_cam_depth_py/2} ${0.019792+0.009}" rpy="-${pi/2} -${pi/2} 0" />
+            <origin xyz="0 ${0.10485-d415_cam_depth_py/2} ${0.019792+0.00945}" rpy="-${pi/2} -${pi/2} 0" />
         </xacro:sensor_d415>
         <link name="onrobot_eyes_base_link"/>

Commit message: Updated camera transform

File: workspace/src/par_pkg/urdf/onrobot_eyes.xacro (robot description, xacro)
@@ -20,5 +20,5 @@
             industrial_calibration seems like a good package for doing this.
         -->
-            <origin xyz="0 ${0.10485-d415_cam_depth_py/2} ${0.019792+0.00945}" rpy="-${pi/2} -${pi/2} 0" />
+            <origin xyz="-0.003 ${(0.10485-d415_cam_depth_py/2) - 0.006} ${0.019792+0.00945}" rpy="-${pi/2} -${pi/2} 0" />
         </xacro:sensor_d415>
         <link name="onrobot_eyes_base_link"/>

Commit message: Removed y offset for camera

File: workspace/src/par_pkg/urdf/onrobot_eyes.xacro (robot description, xacro)
@@ -20,5 +20,5 @@
             industrial_calibration seems like a good package for doing this.
         -->
-            <origin xyz="-0.003 ${(0.10485-d415_cam_depth_py/2) - 0.006} ${0.019792+0.00945}" rpy="-${pi/2} -${pi/2} 0" />
+            <origin xyz="-0.003 ${(0.10485-d415_cam_depth_py/2)} ${0.019792+0.00945}" rpy="-${pi/2} -${pi/2} 0" />
         </xacro:sensor_d415>
         <link name="onrobot_eyes_base_link"/>

Commit message: Re-apply macro

File: workspace/src/par_pkg/urdf/onrobot_eyes.xacro (robot description, xacro)
@@ -20,5 +20,5 @@
             industrial_calibration seems like a good package for doing this.
         -->
-            <origin xyz="-0.003 ${(0.10485-d415_cam_depth_py/2)} ${0.019792+0.00945}" rpy="-${pi/2} -${pi/2} 0" />
+            <origin xyz="-0.003 ${(0.10485-d415_cam_depth_py/2) - 0.006} ${0.019792+0.00945}" rpy="-${pi/2} -${pi/2} 0" />
         </xacro:sensor_d415>
         <link name="onrobot_eyes_base_link"/>
