Commit message: Added aliases, better gripper config and driver params

File: workspace/src/par_pkg/srdf/arm-with-camera-gripper.srdf.xacro (robot description, xacro)
@@ -12,11 +12,12 @@
     <disable_collisions link1="right_inner_finger" link2="right_inner_knuckle" reason="Adjacent" />
     <disable_collisions link1="right_inner_finger" link2="right_outer_knuckle" reason="Adjacent" />
-    <disable_collisions link1="right_outer_finger" link2="right_inner_knuckle" reason="Adjacent" />
+    <disable_collisions link1="right_inner_knuckle" link2="right_outer_knuckle" reason="Never" />
     <disable_collisions link1="left_inner_finger" link2="left_inner_knuckle" reason="Adjacent" />
     <disable_collisions link1="left_inner_finger" link2="left_outer_knuckle" reason="Adjacent" />
-    <disable_collisions link1="left_outer_finger" link2="left_inner_knuckle" reason="Adjacent" />
-    <disable_collisions link1="onrobot_rg2_base_link" link2="right_outer_knuckle" reason="Never" />
-    <disable_collisions link1="onrobot_rg2_base_link" link2="right_inner_knuckle" reason="Never" />
-    <disable_collisions link1="onrobot_rg2_base_link" link2="left_outer_knuckle" reason="Never" />
-    <disable_collisions link1="onrobot_rg2_base_link" link2="left_inner_knuckle" reason="Never" />
+    <disable_collisions link1="left_inner_knuckle" link2="left_outer_knuckle" reason="Never" />
+    <disable_collisions link1="left_inner_finger" link2="right_inner_finger" reason="Never" />
+    <disable_collisions link1="onrobot_rg2_base_link" link2="right_outer_knuckle" reason="Adjacent" />
+    <disable_collisions link1="onrobot_rg2_base_link" link2="right_inner_knuckle" reason="Adjacent" />
+    <disable_collisions link1="onrobot_rg2_base_link" link2="left_outer_knuckle" reason="Adjacent" />
+    <disable_collisions link1="onrobot_rg2_base_link" link2="left_inner_knuckle" reason="Adjacent" />
 </robot>

File: workspace/src/par_pkg/urdf/arm-with-camera.urdf.xacro (robot description, xacro)
@@ -4,10 +4,9 @@
     <xacro:arg name="ur_type" default="ur5x"/>
     <xacro:include filename="$(find ur_description)/urdf/ur.urdf.xacro"/>
-    <xacro:include filename="onrobot_rg2_model.urdf"/>
     <xacro:include filename="onrobot_quick_changer_model.urdf"/>
     <xacro:include filename="onrobot_eyes_model.urdf"/>
     <xacro:macro name="ur" params="name ur_type"/>
     <joint name="eyes_joint" type="fixed">
-        <origin rpy="0 0 3.1416" xyz="0 0 0"/>
+        <origin rpy="0 0 ${pi}" xyz="0 0 0"/>
         <parent link="tool0"/>
         <child link="onrobot_eyes_base_link"/>
@@ -15,14 +14,8 @@
     </joint>
     <joint name="quick_changer_joint" type="fixed">
-        <origin rpy="0 0 1.5708" xyz="0 0 0"/>
+        <origin rpy="0 0 ${pi/2}" xyz="0 0 0"/>
         <parent link="onrobot_eyes_tool_link"/>
         <child link="onrobot_quick_changer_base_link"/>
         <axis xyz="0 0 0"/>
     </joint>
-    <joint name="gripper_joint" type="fixed">
-        <origin rpy="0 0 0" xyz="0 0 0"/>
-        <parent link="onrobot_quick_changer_tool_link"/>
-        <child link="onrobot_rg2_base_link"/>
-        <axis xyz="0 0 0"/>
-    </joint>
 </robot>

File: workspace/src/par_pkg/urdf/onrobot_rg2_model.urdf (robot description, URDF)
Before this commit: robot onrobot_rg2_model, 7 links, 6 joints
Links:
- link onrobot_rg2_base_link: geometry collision mesh filename=package://par_pkg/meshes/collision/base_link.stl; visual mesh filename=package://par_pkg/meshes/visual/base_link_v2.stl

Commit message: Updated camera urdf to get camera baselink

File: workspace/src/par_pkg/srdf/arm-with-camera-gripper.srdf.xacro (robot description, xacro)
@@ -3,9 +3,5 @@
     <xacro:arg name="name" default="ur" />
     <xacro:arg name="prefix" default="" />
-    <xacro:include filename="$(find ur_moveit_config)/srdf/ur.srdf.xacro" />
-    <xacro:macro name="ur_srdf" params="name prefix"/>
-    <xacro:ur_srdf name="$(arg name)" prefix="$(arg prefix)" />
-    <disable_collisions link1="wrist_3_link" link2="onrobot_eyes_base_link" reason="Adjacent" />
-    <disable_collisions link1="onrobot_eyes_base_link" link2="onrobot_quick_changer_base_link" reason="Adjacent" />
+    <xacro:include filename="arm-with-camera.srdf.xacro"/>
     <disable_collisions link1="onrobot_eyes_base_link" link2="onrobot_rg2_base_link" reason="Never" />
     <disable_collisions link1="onrobot_quick_changer_base_link" link2="onrobot_rg2_base_link" reason="Adjacent" />

File: workspace/src/par_pkg/srdf/arm-with-camera.srdf.xacro (robot description, xacro)
@@ -8,3 +8,4 @@
     <disable_collisions link1="wrist_3_link" link2="onrobot_eyes_base_link" reason="Adjacent" />
     <disable_collisions link1="onrobot_eyes_base_link" link2="onrobot_quick_changer_base_link" reason="Adjacent" />
+    <disable_collisions link1="camera_link" link2="onrobot_eyes_base_link" reason="Never" />
 </robot>

File: workspace/src/par_pkg/urdf/arm-with-camera-gripper.urdf.xacro (robot description, xacro)
@@ -3,21 +3,6 @@
     <xacro:arg name="name" default="ur"/>
     <xacro:arg name="ur_type" default="ur5x"/>
-    <xacro:include filename="$(find ur_description)/urdf/ur.urdf.xacro"/>
+    <xacro:include filename="arm-with-camera.urdf.xacro"/>
     <xacro:include filename="onrobot_rg2_model.urdf"/>
-    <xacro:include filename="onrobot_quick_changer_model.urdf"/>
-    <xacro:include filename="onrobot_eyes_model.urdf"/>
-    <xacro:macro name="ur" params="name ur_type"/>
-    <joint name="eyes_joint" type="fixed">
-        <origin rpy="0 0 ${pi}" xyz="0 0 0"/>
-        <parent link="tool0"/>
-        <child link="onrobot_eyes_base_link"/>
-        <axis xyz="0 0 0"/>
-    </joint>
-    <joint name="quick_changer_joint" type="fixed">
-        <origin rpy="0 0 ${pi/2}" xyz="0 0 0"/>
-        <parent link="onrobot_eyes_tool_link"/>
-        <child link="onrobot_quick_changer_base_link"/>
-        <axis xyz="0 0 0"/>
-    </joint>
     <joint name="gripper_joint" type="fixed">
         <origin rpy="0 0 0" xyz="0 0 0"/>

File: workspace/src/par_pkg/urdf/arm-with-camera.urdf.xacro (robot description, xacro)
@@ -6,9 +6,15 @@
     <xacro:include filename="onrobot_quick_changer_model.urdf"/>
     <xacro:include filename="onrobot_eyes_model.urdf"/>
-    <!-- <xacro:include filename="$(find realsense2_description)/urdf/_d415.urdf.xacro"/> -->
+    <xacro:include filename="$(find realsense2_description)/urdf/_d415.urdf.xacro"/>
     <xacro:macro name="ur" params="name ur_type"/>
-    <!-- <xacro:sensor_d415 parent="on_robot_eyes_base_link" use_nominal_extrinsics="true" add_plug="false" use_mesh="true">
-        <origin xyz="0 0.105 0" rpy="0 0 0"/>
-    </xacro:sensor_d415> -->
+    <xacro:sensor_d415 parent="onrobot_eyes_base_link" use_nominal_extrinsics="true" add_plug="false" use_mesh="false">
+        <!--
+            These measurements are not 100% accurate, they're the best
+            I could get based on manually aligning it in blender.
+            We need to preform camera extrinsics calibration manually to get these values.
+            industrial_calibration seems like a good package for doing this.
+        -->
+        <origin xyz="-0.000473 0.093319 0.021695" rpy="-${pi/2} -${pi/2} 0"/>
+    </xacro:sensor_d415>
     <joint name="eyes_joint" type="fixed">
         <origin rpy="0 0 ${pi}" xyz="0 0 0"/>

File: workspace/src/par_pkg/urdf/onrobot_eyes_model.urdf (robot description, URDF)
Before this commit: robot onrobot_eyes_model, 3 links, 2 joints
Links:
- removed link camera_link
Joints:
- removed joint camera_joint
