Commit message: Added the mounting plate to the urdf

File: workspace/src/par_pkg/srdf/arm-with-camera.srdf.xacro (robot description, xacro)
@@ -9,3 +9,4 @@
     <disable_collisions link1="onrobot_eyes_base_link" link2="onrobot_quick_changer_base_link" reason="Adjacent" />
     <disable_collisions link1="camera_link" link2="onrobot_eyes_base_link" reason="Never" />
+    <disable_collisions link1="base_link" link2="mount_link" reason="Adjacent"/>
 </robot>

File: workspace/src/par_pkg/urdf/arm-with-camera.urdf.xacro (robot description, xacro)
@@ -7,4 +7,6 @@
     <xacro:include filename="onrobot_eyes.urdf"/>
     <xacro:include filename="$(find realsense2_description)/urdf/_d415.urdf.xacro"/>
+    <xacro:property name="plate_depth" value="0.0127" />
+    <xacro:property name="plate_size" value="0.30"/>
     <xacro:macro name="ur" params="name ur_type"/>
     <xacro:sensor_d415 parent="onrobot_eyes_base_link" use_nominal_extrinsics="true" add_plug="false" use_mesh="false">
@@ -25,4 +27,29 @@
         <axis xyz="0 0 0"/>
     </joint>
+    <link name="mount_link">
+        <visual>
+            <origin xyz="0 0 ${plate_depth/2}"/>
+            <geometry>
+                <box size="${plate_size} ${plate_size} ${plate_depth}" />
+            <geometry/>
+        </visual>
+        <collision>
+        <origin xyz="0 0 ${plate_depth/2}"/>
+            <geometry>
+                <box size="${plate_size} ${plate_size} ${plate_depth}" />
+            <geometry/>
+        </collision>
+    </link>
+    <joint name="world_joint" type="fixed">
+        <parent link="world"/>
+        <child link="mount_link"/>
+        <axis xyz="0 0 0"/>
+    </joint>
+    <joint name="mount_joint" type="fixed">
+        <origin xyz="0 0 ${plate_depth}"/>
+        <parent link="mount_link"/>
+        <child link="base_link"/>
+        <axis xyz="0 0 0"/>
+    </joint>
     <joint name="eyes_joint" type="fixed">
         <origin rpy="0 0 ${pi}" xyz="0 0 0"/>
