Commit message: Moved all rg2 stuff into its own packages, included ur drivers

File: workspace/src/onrobot_rg2_description/urdf/onrobot_rg2_macro.xacro (robot description, xacro)
@@ -21,10 +21,10 @@
             <visual>
                 <geometry>
-                    <mesh filename="package://par_pkg/meshes/visual/rg2_base_link${poly}.dae" />
+                    <mesh filename="package://onrobot_rg2_description/meshes/visual/rg2_base_link${poly}.dae" />
                 </geometry>
             </visual>
             <collision>
                 <geometry>
-                    <mesh filename="package://par_pkg/meshes/collision/rg2_base_link.stl" />
+                    <mesh filename="package://onrobot_rg2_description/meshes/collision/rg2_base_link.stl" />
                 </geometry>
             </collision>
@@ -33,10 +33,10 @@
             <visual>
                 <geometry>
-                    <mesh filename="package://par_pkg/meshes/visual/rg2_outer_knuckle${poly}.dae" />
+                    <mesh filename="package://onrobot_rg2_description/meshes/visual/rg2_outer_knuckle${poly}.dae" />
                 </geometry>
             </visual>
             <collision>
                 <geometry>
-                    <mesh filename="package://par_pkg/meshes/collision/rg2_outer_knuckle.stl" />
+                    <mesh filename="package://onrobot_rg2_description/meshes/collision/rg2_outer_knuckle.stl" />
                 </geometry>
             </collision>
@@ -45,10 +45,10 @@
             <visual>
                 <geometry>
-                    <mesh filename="package://par_pkg/meshes/visual/rg2_inner_knuckle${poly}.dae" />
+                    <mesh filename="package://onrobot_rg2_description/meshes/visual/rg2_inner_knuckle${poly}.dae" />
                 </geometry>
             </visual>
             <collision>
                 <geometry>
-                    <mesh filename="package://par_pkg/meshes/collision/rg2_inner_knuckle.stl" />
+                    <mesh filename="package://onrobot_rg2_description/meshes/collision/rg2_inner_knuckle.stl" />
                 </geometry>
             </collision>
@@ -57,10 +57,10 @@
             <visual>
                 <geometry>
-                    <mesh filename="package://par_pkg/meshes/visual/rg2_finger${poly}.dae" />
+                    <mesh filename="package://onrobot_rg2_description/meshes/visual/rg2_finger${poly}.dae" />
                 </geometry>
             </visual>
             <collision>
                 <geometry>
-                    <mesh filename="package://par_pkg/meshes/collision/rg2_finger.stl" />
+                    <mesh filename="package://onrobot_rg2_description/meshes/collision/rg2_finger.stl" />
                 </geometry>
             </collision>
@@ -69,10 +69,10 @@
             <visual>
                 <geometry>
-                    <mesh filename="package://par_pkg/meshes/visual/rg2_outer_knuckle${poly}.dae" />
+                    <mesh filename="package://onrobot_rg2_description/meshes/visual/rg2_outer_knuckle${poly}.dae" />
                 </geometry>
             </visual>
             <collision>
                 <geometry>
-                    <mesh filename="package://par_pkg/meshes/collision/rg2_outer_knuckle.stl" />
+                    <mesh filename="package://onrobot_rg2_description/meshes/collision/rg2_outer_knuckle.stl" />
                 </geometry>
             </collision>
@@ -81,10 +81,10 @@
             <visual>
                 <geometry>
-                    <mesh filename="package://par_pkg/meshes/visual/rg2_inner_knuckle${poly}.dae" />
+                    <mesh filename="package://onrobot_rg2_description/meshes/visual/rg2_inner_knuckle${poly}.dae" />
                 </geometry>
             </visual>
             <collision>
                 <geometry>
-                    <mesh filename="package://par_pkg/meshes/collision/rg2_inner_knuckle.stl" />
+                    <mesh filename="package://onrobot_rg2_description/meshes/collision/rg2_inner_knuckle.stl" />
                 </geometry>
             </collision>
@@ -93,10 +93,10 @@
             <visual>
                 <geometry>
-                    <mesh filename="package://par_pkg/meshes/visual/rg2_finger${poly}.dae" />
+                    <mesh filename="package://onrobot_rg2_description/meshes/visual/rg2_finger${poly}.dae" />
                 </geometry>
             </visual>
             <collision>
                 <geometry>
-                    <mesh filename="package://par_pkg/meshes/collision/rg2_finger.stl" />
+                    <mesh filename="package://onrobot_rg2_description/meshes/collision/rg2_finger.stl" />
                 </geometry>
             </collision>

File: workspace/src/par_pkg/srdf/ur_assembly.srdf.xacro (robot description, xacro)
@@ -7,4 +7,5 @@
     <xacro:arg name="prefix" default="" />
     <xacro:include filename="$(find ur_moveit_config)/srdf/ur_macro.srdf.xacro" />
+    <xacro:include filename="$(find onrobot_rg2_description)/srdf/onrobot_rg2.srdf.xacro" />
     <xacro:property name="ik_group" value="$(arg prefix)$(arg name)_manipulator_end_effector"/>
     <xacro:ur_srdf name="$(arg name)" prefix="$(arg prefix)" />
@@ -21,4 +22,5 @@
     <disable_collisions link1="base_link_inertia" link2="mount_plate_link" reason="Adjacent" />
     <xacro:if value="$(arg gripper)">
+        <xacro:rg2_srdf parent="onrobot_quick_changer_base_link"/>
         <group name="${ik_group}">
             <chain base_link="$(arg prefix)base_link" tip_link="end_effector_link"/>
@@ -29,19 +31,4 @@
         <disable_collisions link1="onrobot_quick_changer_base_link" link2="onrobot_rg2_base_link"
             reason="Adjacent" />
-        <disable_collisions link1="right_finger" link2="right_inner_knuckle" reason="Adjacent" />
-        <disable_collisions link1="right_finger" link2="right_outer_knuckle" reason="Adjacent" />
-        <disable_collisions link1="right_inner_knuckle" link2="right_outer_knuckle" reason="Never" />
-        <disable_collisions link1="left_finger" link2="left_inner_knuckle" reason="Adjacent" />
-        <disable_collisions link1="left_finger" link2="left_outer_knuckle" reason="Adjacent" />
-        <disable_collisions link1="left_inner_knuckle" link2="left_outer_knuckle" reason="Never" />
-        <disable_collisions link1="left_finger" link2="right_finger" reason="Never" />
-        <disable_collisions link1="onrobot_rg2_base_link" link2="right_outer_knuckle"
-            reason="Adjacent" />
-        <disable_collisions link1="onrobot_rg2_base_link" link2="right_inner_knuckle"
-            reason="Adjacent" />
-        <disable_collisions link1="onrobot_rg2_base_link" link2="left_outer_knuckle"
-            reason="Adjacent" />
-        <disable_collisions link1="onrobot_rg2_base_link" link2="left_inner_knuckle"
-            reason="Adjacent" />
     </xacro:if>
     <xacro:unless value="$(arg gripper)">

File: workspace/src/par_pkg/urdf/ur_assembly_macro.xacro (robot description, xacro)
@@ -4,5 +4,5 @@
     <xacro:include filename="$(find par_pkg)/urdf/onrobot_eyes.xacro" />
     <xacro:include filename="$(find par_pkg)/urdf/onrobot_quick_changer.xacro" />
-    <xacro:include filename="$(find par_pkg)/urdf/onrobot_rg2.xacro" />
+    <xacro:include filename="$(find onrobot_rg2_description)/urdf/onrobot_rg2_macro.xacro" />
     <xacro:property name="mount_plate_size" value="0.194" />
     <xacro:property name="mount_plate_depth" value="0.0127" />
